File: tektronix_465_original/tektronix_465_original.kicad_sch (KiCad schematic)
At the start: 0 parts

Commit message: Added sheets for original scopes high level block diagram
Other:
- added sheet calibrator (calibrator.kicad_sch)
- added sheet ch1_preamp (ch1_preamp.kicad_sch)
- added sheet fan_motor (fan_motor.kicad_sch)
- added sheet horizontal_amp (horizontal_amp.kicad_sch)
- added sheet lowvoltage_psu (lowvoltage_psu.kicad_sch)
- added sheet sweep_control_and_z_axis_logic (sweep_control_and_z_axis_logic.kicad_sch)
- added sheet trigger_generator_A (untitled.kicad_sch)
- added sheet trigger_view_amp (trigger_view_amp.kicad_sch)
- added sheet vertical_output_amp (vertical_output_amp.kicad_sch)
- added sheet vertical_switching (vertical_switching.kicad_sch)
- added sheet z_axis_amp (z_axis_amp.kicad_sch)
