File: tektronix_465_original/ch1_preamp.kicad_sch (KiCad schematic)
At the start: 0 parts

Commit message: tekOG, started on the CH1 preamp section
Parts:
- added C1: 0.25-1.5, symbol Device:C_Variable
- added C18: 3.9, symbol Device:C_Polarized
- added C2: SEL, symbol Device:C_Polarized
- added C21: 0.22, symbol Device:C_Polarized
- added C22: 300, symbol Device:C_Polarized
- added C23: 6.8uF, symbol Device:C_Polarized
- added C25, C36, C39: 0.02, symbol Device:C
- added C27: 2-18, symbol Device:C_Trim
- added C3: C_Polarized, symbol Device:C_Polarized
- added C32: 6.8uF, symbol Device:C
- added C33: 1-4, symbol Device:C_Trim
- added C34: 150, symbol Device:C
- added C37: 0.001, symbol Device:C_Polarized
- added C38: 0.001, symbol Device:C
- added C4: 0.005, symbol Device:C
- added D18: (CR18)SE365, symbol Device:D
- added D18: (CR18)8.7V, symbol Device:D_Zener
- added D21: (VR21), symbol Device:D_Zener
- added D31, D32: 1N4152, symbol Device:D
- added J1: Conn_Coaxial, symbol Connector:Conn_Coaxial
- added J2: Conn_Coax_extra, symbol Connector:Conn_01x01_Pin
- added Q20: 2N5911/2N5912, Package_TO_SOT_THT:TO-78-6, symbol techtronix_lib:2N5911/2N5912
- added Q32, Q36: NPN, symbol Simulation_SPICE:NPN
- added Q382: MPS-A65, symbol Simulation_SPICE:PNP
- added Q386: 2N2907A, symbol Simulation_SPICE:PNP
- added Q42, Q44 (x2): PNP, symbol Simulation_SPICE:PNP
- added R1: 51, symbol Device:R
- added R15, R4: 1M, symbol Device:R
- added R16: 470k, symbol Device:R
- added R18: 330, symbol Device:R
- added R21, R27: 150, symbol Device:R
- added R22, R23: 20, symbol Device:R
- added R26: 12k, symbol Device:R
- added R3: 4.7, symbol Device:R
- added R32, R36: 1.43k, symbol Device:R
- added R33: 100, symbol Device:R
- added R34, R35, R44: R, symbol Device:R
- added R37, R38: 620, symbol Device:R
- added R41, R43: 931, symbol Device:R
- added R45 (x2): 102, symbol Device:R
- added RV25: 5k, symbol Device:R_Potentiometer
- added SW1, SW11, SW2, SW5, SW7, SW9: SW_Push, symbol Switch:SW_Push
- added SW10, SW12, SW3, SW4, SW6, SW8: SW_Push_Open, symbol Switch:SW_Push_Open
Connections:
- new net: Q44.1 (C), R45.1
- new net: C38.2, Q44.3 (E), R38.2, R43.1
- new net: R3.2, R4.1, SW1.1, SW3.1 (A)
- new net: SW1.2, SW3.2 (B), SW4.1 (A)
- new net: R4.2, SW2.2, SW4.2 (B)
- new net: C4.2, D18.1 (K), Q20.3 (G), R16.2, R18.1
- new net: C37.1, Q42.3 (E), R37.1, R41.2
- new net: C37.2, Q32.1 (C), R37.2
- new net: C38.1, Q36.1 (C), R38.1
- new net: R15.1, SW12.2 (B)
- new net: C33.1, R33.1
- new net: C33.2, R33.2
- new net: C18.1, R18.2
- new net: C27.1, Q36.2 (B), R26.2, R27.1
- new net: SW10.1 (A), SW7.2, SW8.2 (B), SW9.1
- new net: SW10.2 (B), SW12.1 (A)
- new net: R26.1, RV25.2
- new net: C22.1, Q20.2 (D), R22.1
- new net: C22.2, D31.1 (K), D32.2 (A), Q20.5 (S), Q32.2 (B), R22.2
- new net: Q32.3 (E), Q36.3 (E)
- new net: SW6.2 (B), SW8.1 (A)
- new net: C3.1, R3.1
- new net: Q20.6 (D), R23.1
- new net: C1.1, C2.1, C3.2, R1.2
- new net: Q42.1 (C), R44.2
- new net: C4.1, R16.1, SW11.2
- new net: D21.2 (A), R21.1
- new net: Q20.1 (S), R21.2
- new net -8V: C23.2, C25.1, D18.2 (A), Q20.7 (G), R23.2, RV25.3
- new net CH1_INPUT: J1.1 (In), R1.1
- new net CH1_ScaleFactor: J2.1 (Pin_1)
- new net Earth: C1.2, C18.2, C2.2, C21.2, C23.1, C25.2, C27.2, D31.2 (A), D32.1 (K), J1.2 (Ext), R15.2, R27.2, SW2.1
- new net P,+15: C21.1, D21.1 (K), R41.1, R43.2, RV25.1
Other:
- note added: "CH1 or X (BNC Connector with shield pin)"

Commit message: completed most of ch1 vertitical preamp
Parts:
- removed D18: (CR18)8.7V, symbol Device:D_Zener
- removed Q20: 2N5911/2N5912, Package_TO_SOT_THT:TO-78-6, symbol techtronix_lib:2N5911/2N5912
- removed Q44: PNP, symbol Simulation_SPICE:PNP
- removed R45: 102, symbol Device:R
- added C107, C109: 0.001, symbol Device:C
- added C42: 0.02, symbol Device:C
- added C48: 2-18, symbol Device:C_Trim
- added C49: 12, symbol Device:C
- added C5: C_Trim, symbol Device:C_Trim
- added C6: C, symbol Device:C
- added JP1, JP2: Jumper_2_Bridged, symbol Jumper:Jumper_2_Bridged
- added Q102, Q104: NPN, symbol Simulation_SPICE:NPN
- added Q20: 2N5911/2N5912, Package_TO_SOT_THT:TO-78-6, symbol techtronix_lib:2N5911/2N5912(v2)
- added R106, R108: 300, symbol Device:R
- added R107, R109: 27, symbol Device:R
- added R2: R_Trim, symbol Device:R_Trim
- added R39, R42: 100, symbol Device:R
- added R48: 1k, symbol Device:R_Trim
- added R49: 66.5, symbol Device:R
- added R5, R6, R7, R8: R, symbol Device:R
- added RV1: R_Potentiometer, symbol Device:R_Potentiometer
- added SW13, SW14: SW_Push, symbol Switch:SW_Push
- added TH1: Thermistor_NTC, symbol Device:Thermistor_NTC
- R35: value R -> 100k
- R44: value R -> 102
Connections:
- net -8V: now also C32.1, C36.1, R32.2, R36.2, Q20.7 (G2)
- net Earth: now also C32.2, C36.2, C39.1, R44.2, R45.2, C42.2
- net at Q44.1 (C), R45.1: now also JP2.1 (A), Q104.2 (B)
- net at Q44.2 (B): now also Q42.2 (B), R42.2
- net at R4.2, SW2.2, SW4.2 (B): now also SW5.1, SW6.1 (A)
- net at C4.2, D18.1 (K), R16.2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: now also Q20.3 (G1)
- net at C33.1, R33.1: now also C34.2, Q32.3 (E), R32.1
- net at C33.2, R33.2: now also Q36.3 (E), R36.1
- net at C22.1, R22.1: now also D31.1 (K), D32.2 (A), Q32.2 (B), Q20.2 (D1)
- net at C34.1: now also R34.2, R35.2
- net at C39.2: now also R39.2
- net at R23.1: now also Q20.6 (D2)
- net at Q42.1 (C): now also R44.1, JP1.2 (B), Q102.2 (B); no longer R44.2
- net CH1_ATTEN_OUT: now reaches C4.1, R16.1, SW11.2
- net at R21.2: now also Q20.1 (S1)
- net P,+5: now reaches R34.1
- net P,+5: now also C42.1, R42.1
- net TO_R85(2): now reaches R35.1
- new net: C49.1, JP1.1 (A), R48.1, R49.1, SW13.1
- new net: C109.1, Q104.3 (E), R108.1
- new net: C109.2, R109.1
- new net: C5.1, C6.1, R5.1, SW13.2
- new net: C6.2, JP2.2 (B), R2.2, R5.2, SW14.1
- new net: R108.2, R109.2
- new net: C22.2, Q20.5 (S2), R22.2
- new net: C107.1, Q102.1 (C), R106.1
- new net: R106.2, R107.2
- new net: C48.1, R48.2
- new net: C48.2, C49.2, R49.2, SW14.2
- new net: Q102.3 (E), Q104.1 (C)
- new net: C107.2, R107.1
- new net: C5.2, R2.1
- new net +55V: R39.1
Other:
- note added: "Board to Board Coupling"
- note added: "Partial A1 CH1 Atten Board"
- moved on the sheet: C18, C21, C22, C23, C25, C27, C32, C33, C34, C36, C37, C38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
